File: esp-drone.sch (KiCad schematic (older format))
At the start: 5 parts, among them U1 USB_C_16_PIN

Commit message: .
Parts:
- added C? (x2): 1uF, symbol Device:C
- added C?: 10uF, symbol Device:C
- added D?: BAT60B, symbol Device:D
- added J?: Conn_01x02, symbol Connector_Generic:Conn_01x02
- added Q?: AO3401A, Package_TO_SOT_SMD:SOT-23, symbol Transistor_FET:AO3401A
- added R?: 200R, symbol Device:R
- added R? (x2): 10K, symbol Device:R
- added R?: 10uF, symbol Device:R
- added R? (x3): 82K, symbol Device:R
- added U?: BC847BDW1T1G, Package_TO_SOT_SMD:SOT-363_SC-70-6, symbol esp-drone:BC847BDW1T1G
- added U?: ME6211C33M5G-N, Package_TO_SOT_SMD:SOT-23-5, symbol LDO:ME6211C33M5G-N
Connections:
- net CP_DTR: now also R?.2, U?.1 (E2)
- net CP_RTS: now also R?.1, U?.4 (E1)
- net CP_TXD: now also R?.1; no longer U?.26 (TXD)
- net GND: now also C?.2, C?.2, C?.2, J?.2 (Pin_2), R?.2, R?.2, R?.2, U?.2 (GND)
- net VBUS: now also D?.2 (A), Q?.1 (G), R?.1
- new net: R?.2, U?.26 (TXD)
- new net: R?.2, U?.2 (B2)
- new net: R?.1, U?.5 (B1)
- new net +3V3: C?.1, C?.1, U?.5 (VOUT)
- new net +BATT: J?.1 (Pin_1), Q?.3 (D), R?.1, R?.1
- new net ADC_BAT: R?.1, R?.2
- new net ESP_EN: U?.3 (C1)
- new net ESP_IO0: U?.6 (C2)
- new net VSS: C?.1, D?.1 (K), Q?.2 (S), U?.1 (VIN), U?.3 (EN)

Commit message: sch finish
Parts:
- added AE1: Antenna, Antenna:CA-C03, symbol Device:Antenna
- added C1: 10nF, Capacitor_SMD:C_0402_1005Metric, symbol Device:C
- added C10, C11, C12, C13, C15, C16, C17, C18, C2, C4, C7, C8: 0.1uF, Capacitor_SMD:C_0402_1005Metric, symbol Device:C
- added C14, C19, C20: 10uF, Capacitor_SMD:C_0402_1005Metric, symbol Device:C
- added C5: 2.2nF, Capacitor_SMD:C_0402_1005Metric, symbol Device:C
- added D1: LED-WHT, LED_SMD:LED_0402_1005Metric, symbol Device:LED
- added D2: LED-BLE, LED_SMD:LED_0402_1005Metric, symbol Device:LED
- added D3: LED-RED, LED_SMD:LED_0402_1005Metric, symbol Device:LED
- added D4: LED-GRN, LED_SMD:LED_0402_1005Metric, symbol Device:LED
- added D6, D7, D8, D9: 1N4148WT, Diode_SMD:D_SOD-523, symbol Diode:1N4148WT
- added ESP1: ESP32PICO_D4, SOC:ESP32_PICO_D4, symbol SOC:ESP32PICO_D4
- added FB1: 330R at 100MHz, Resistor_SMD:R_0402_1005Metric, symbol Device:Ferrite_Bead
- added J10, J11, J6, J7: Conn_01x02, Connector_JST:JST_PH_S2B-PH-K_1x02_P2.00mm_Horizontal, symbol Connector_Generic:Conn_01x02
- added J12: Conn_01x26, Connector_FFC-FPC:TE_2-1734839-4_1x24-1MP_P0.5mm_Horizontal, symbol Connector_Generic:Conn_01x26
- added J2, J3, J8, J9: Conn_01x02, esp-drone:MOTOR_CONN, symbol Connector_Generic:Conn_01x02
- added J4, J5: Conn_01x08, Connector_PinHeader_2.54mm:PinHeader_1x08_P2.54mm_Vertical_SMD_Pin1Right, symbol Connector_Generic:Conn_01x08
- added Q2, Q3, Q4, Q5: AO3400A, Package_TO_SOT_SMD:SOT-23, symbol Transistor_FET:AO3400A
- added R10, R14, R15, R16, R18, R19, R21, R22, R23, R24, R25, R26, R27, R28, R7: 10K, Resistor_SMD:R_0402_1005Metric, symbol Device:R
- added R20: 0R, Resistor_SMD:R_0402_1005Metric, symbol Device:R
- added R8: 2K, Resistor_SMD:R_0402_1005Metric, symbol Device:R
- added R9: 3K, Resistor_SMD:R_0402_1005Metric, symbol Device:R
- added SW1, SW2: SW_MEC_5E, Button:SKSC_NO_HOLE, symbol Switch:SW_MEC_5E
- added U3: MPU-6050, Sensor_Motion:InvenSense_QFN-24_4x4mm_P0.5mm, symbol Sensor_Motion:MPU-6050
- added U6: ESP-PSRAM32, Package_SO:SOIC-8_3.9x4.9mm_P1.27mm, symbol Memory_RAM:ESP-PSRAM32
- added U7: ME6211C28M5G-N, Package_TO_SOT_SMD:SOT-23-5, symbol LDO:ME6211C28M5G-N
- added U8: ME6211C15M5G-N, Package_TO_SOT_SMD:SOT-23-5, symbol LDO:ME6211C15M5G-N
- C3, C6, C9: renamed from C?; footprint (none) -> Capacitor_SMD:C_0402_1005Metric
- D5: renamed from D?; footprint (none) -> Diode_SMD:D_SOD-323
- J1: renamed from J?; footprint (none) -> Connector_JST:JST_XH_S2B-XH-A-1_1x02_P2.50mm_Horizontal
- R1, R11, R12, R13, R17, R2, R3, R4, R5, R6: renamed from R?; footprint (none) -> Resistor_SMD:R_0402_1005Metric
- gave numbers to parts that had none: 4
- renumbered U1 to U2
Connections:
- net +3V3: now also C1.2, C2.1, FB1.1, J4.1 (Pin_1), R14.1, R15.1, R16.1, U3.13 (VDD), U3.8 (VDDIO)
- net +BATT: now also D6.1 (K), D7.1 (K), D8.1 (K), D9.1 (K), J10.2 (Pin_2), J11.2 (Pin_2), J2.2 (Pin_2), J3.2 (Pin_2), J6.1 (Pin_1), J7.1 (Pin_1), J8.2 (Pin_2), J9.2 (Pin_2)
- net CP_RXD: now also ESP1.41 (U0TXD)
- net CP_TXD: now also ESP1.40 (U0RXD)
- net ESP_EN: now also C15.2, C8.1, ESP1.9 (EN), R24.1, SW2.4 (A)
- net ESP_IO0: now also C7.1, ESP1.23 (IO0), SW1.4 (A)
- net GND: now also C1.1, C11.2, C12.2, C13.1, C14.1, C15.1, C16.1, C17.2, C18.2, C19.2, C2.2, C20.2, C4.1, C5.2, C7.2, C8.2, ESP1.49 (GND), J12.15 (Pin_15), J4.4 (Pin_4), J5.5 (Pin_5), Q2.2 (S), Q3.2 (S), Q4.2 (S), Q5.2 (S), R10.1, R18.2, R19.2, R20.2, R21.2, R22.2, R23.2, R7.1, R8.1, R9.1, SW1.1, SW2.1, U3.1 (CLKIN), U3.11 (FSYNC), U3.18 (GND), U3.9 (AD0), U6.4 (VSS), U7.2 (GND), U8.2 (GND)
- net VSS: now also C17.1, C18.1, D1.2 (A), U7.1 (VIN), U7.3 (EN), U8.1 (VIN), U8.3 (EN)
- new net: C4.2, U3.10 (REGOUT)
- new net: C5.1, U3.20 (CPOUT)
- new net: D7.2 (A), J3.1 (Pin_1), J7.2 (Pin_2), Q3.3 (D)
- new net: D6.2 (A), J2.1 (Pin_1), J6.2 (Pin_2), Q2.3 (D)
- new net: D8.2 (A), J10.1 (Pin_1), J8.1 (Pin_1), Q4.3 (D)
- new net: D9.2 (A), J11.1 (Pin_1), J9.1 (Pin_1), Q5.3 (D)
- new net: D1.1 (K), R7.2
- new net: D2.1 (K), R8.2
- new net: D3.1 (K), R9.2
- new net: D4.1 (K), R10.2
- new net: AE1.1 (A), ESP1.2 (LNA_IN)
- new net: J12.8 (Pin_8), R23.1
- new net +1V5: C12.1, C20.1, J12.10 (Pin_10), U8.5 (VOUT)
- new net +2V8: C10.1, C11.1, C19.1, J12.11 (Pin_11), J12.4 (Pin_4), U7.5 (VOUT)
- new net AUX_SCL: J4.5 (Pin_5), R15.2, U3.7 (AUX_SCL)
- new net AUX_SDA: J4.6 (Pin_6), R16.2, U3.6 (AUX_SDA)
- new net BUZ_1: J4.8 (Pin_8)
- new net BUZ_2: J4.7 (Pin_7)
- new net CAM_HREF: J12.9 (Pin_9)
- new net CAM_PCLK: J12.17 (Pin_17)
- new net CAM_RESET: J12.6 (Pin_6)
- new net CAM_VSYNC: J12.7 (Pin_7)
- new net CAM_XCLK: J12.13 (Pin_13)
- new net CAM_Y2: J12.19 (Pin_19)
- new net CAM_Y3: J12.21 (Pin_21)
- new net CAM_Y4: J12.22 (Pin_22)
- new net CAM_Y5: J12.20 (Pin_20)
- new net CAM_Y6: J12.18 (Pin_18)
- new net CAM_Y7: J12.16 (Pin_16)
- new net CAM_Y8: J12.14 (Pin_14)
- new net CAM_Y9: J12.12 (Pin_12)
- new net EXT_IO1: J5.8 (Pin_8)
- new net GNDA: C10.2, J12.2 (Pin_2), R20.1
- new net I2C0_SCL: J12.5 (Pin_5), J4.3 (Pin_3), R28.1, U3.23 (SCL)
- new net I2C0_SDA: J12.3 (Pin_3), J4.2 (Pin_2), R27.1, U3.24 (SDA)
- new net I2C1_SCL: J5.7 (Pin_7), R26.1
- new net I2C1_SDA: J5.6 (Pin_6), R25.1
- new net LED_BLE: D2.2 (A)
- new net LED_GRN: D4.2 (A)
- new net LED_RED: D3.2 (A)
- new net MOT3: Q3.1 (G), R19.1
- new net MOT4: Q5.1 (G), R22.1
- new net MOT_1: Q2.1 (G), R18.1
- new net MOT_2: Q4.1 (G), R21.1
- new net MPU_INT: R14.2, U3.12 (INT)
- new net PSRAM_CS: ESP1.29 (SD3), U6.1 (~CE)
- new net SCLK: ESP1.31 (CLK), U6.6 (SCLK)
- new net SIO0: ESP1.33 (SD1), U6.5 (SI/SIO)
- new net SIO1: ESP1.27 (IO17), U6.2 (SO/SIO)
- new net SIO2: ESP1.32 (SD0), U6.3 (SIO2)
- new net SIO3: ESP1.30 (CMD), U6.7 (SIO3)
- new net SPI_CLK: J5.3 (Pin_3)
- new net SPI_CS0: J5.1 (Pin_1)
- new net SPI_MOSI: J5.2 (Pin_2), J5.4 (Pin_4)
- new net VDD33_ESP: C13.2, C14.2, ESP1.1 (VDDA), ESP1.19 (VDD3P3_RTC), ESP1.3 (VDDA3P3), ESP1.37 (VDD3P3_CPU), ESP1.4 (VDDA3P3), ESP1.43 (VDDA), ESP1.46 (VDDA), FB1.2, R24.2, R25.2, R26.2, R27.2, R28.2
- new net VDD_SIO: C16.2, ESP1.26 (VDD_SDIO_NC), U6.8 (VCC)
- no-connect marks 17 -> 30
Other:
- moved on the sheet: C3, C6, C9, D5, J1, Q1, R1, R11, R12, R13, R17, R2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

Commit message: .
Parts:
- removed J2, J3, J8, J9: Conn_01x02, esp-drone:MOTOR_CONN, symbol Connector_Generic:Conn_01x02
Changed lines of the file:
@@
 NoConn ~ 12500 3850
-$Comp
-L Connector_Generic:Conn_01x02 J3
-U 1 1 616E96C7
-P 6550 3400
-F 0 "J3" H 6500 3200 50  0000 L CNN
-F 1 "Conn_01x02" H 6500 3500 50  0000 L CNN
-F 2 "esp-drone:MOTOR_CONN" H 6550 3400 50  0001 C CNN
-F 3 "~" H 6550 3400 50  0001 C CNN
-	1    6550 3400
-	-1   0    0    1
-$EndComp
-$Comp
-L Connector_Generic:Conn_01x02 J2
-U 1 1 616E9D68
-P 6550 1400
-F 0 "J2" H 6500 1200 50  0000 L CNN
-F 1 "Conn_01x02" H 6500 1500 50  0000 L CNN
-F 2 "esp-drone:MOTOR_CONN" H 6550 1400 50  0001 C CNN
-F 3 "~" H 6550 1400 50  0001 C CNN
-	1    6550 1400
-	-1   0    0    1
-$EndComp
-$Comp
-L Connector_Generic:Conn_01x02 J8
-U 1 1 616EA341
-P 8450 1400
-F 0 "J8" H 8400 1200 50  0000 L CNN
-F 1 "Conn_01x02" H 8400 1500 50  0000 L CNN
-F 2 "esp-drone:MOTOR_CONN" H 8450 1400 50  0001 C CNN
-F 3 "~" H 8450 1400 50  0001 C CNN
-	1    8450 1400
-	-1   0    0    1
-$EndComp
-$Comp
-L Connector_Generic:Conn_01x02 J9
-U 1 1 616EAA14
-P 8450 3400
-F 0 "J9" H 8400 3200 50  0000 L CNN
-F 1 "Conn_01x02" H 8400 3500 50  0000 L CNN
-F 2 "esp-drone:MOTOR_CONN" H 8450 3400 50  0001 C CNN
-F 3 "~" H 8450 3400 50  0001 C CNN
-	1    8450 3400
-	-1   0    0    1
-$EndComp
-Wire Wire Line
-	6750 1300 6750 1100
-Wire Wire Line
-	6750 1100 7150 1100
-Wire Wire Line
-	6750 1400 6750 1650
-Wire Wire Line
-	6750 1650 7150 1650
-Wire Wire Line
-	6750 3300 6750 3100
-Wire Wire Line
-	6750 3100 7150 3100
-Wire Wire Line
-	6750 3400 6750 3650
-Wire Wire Line
-	6750 3650 7150 3650
-Wire Wire Line
-	8650 1300 8650 1100
-Wire Wire Line
-	8650 1100 9000 1100
-Wire Wire Line
-	8650 1400 8650 1650
-Wire Wire Line
-	8650 1650 9000 1650
-Wire Wire Line
-	8650 3300 8650 3100
-Wire Wire Line
-	8650 3100 9000 3100
-Wire Wire Line
-	8650 3400 8650 3650
-Wire Wire Line
-	8650 3650 9000 3650
 $Comp
 L Memory_RAM:ESP-PSRAM32 U6

Commit message: .
Parts:
- removed C1: 10nF, Capacitor_SMD:C_0402_1005Metric, symbol Device:C
- removed C10, C11, C12, C16, C17, C18: 0.1uF, Capacitor_SMD:C_0402_1005Metric, symbol Device:C
- removed C19, C20: 10uF, Capacitor_SMD:C_0402_1005Metric, symbol Device:C
- removed C5: 2.2nF, Capacitor_SMD:C_0402_1005Metric, symbol Device:C
- removed J12: Conn_01x26, Connector_FFC-FPC:TE_2-1734839-4_1x24-1MP_P0.5mm_Horizontal, symbol Connector_Generic:Conn_01x26
- removed R14, R15, R16, R23: 10K, Resistor_SMD:R_0402_1005Metric, symbol Device:R
- removed R20: 0R, Resistor_SMD:R_0402_1005Metric, symbol Device:R
- removed U3: MPU-6050, Sensor_Motion:InvenSense_QFN-24_4x4mm_P0.5mm, symbol Sensor_Motion:MPU-6050
- removed U6: ESP-PSRAM32, Package_SO:SOIC-8_3.9x4.9mm_P1.27mm, symbol Memory_RAM:ESP-PSRAM32
- removed U7: ME6211C28M5G-N, Package_TO_SOT_SMD:SOT-23-5, symbol LDO:ME6211C28M5G-N
- removed U8: ME6211C15M5G-N, Package_TO_SOT_SMD:SOT-23-5, symbol LDO:ME6211C15M5G-N
- added C3: 0.1uF, Capacitor_SMD:C_0402_1005Metric, symbol Device:C
- added R3: 10K, Resistor_SMD:R_0402_1005Metric, symbol Device:R
- added U3: ICM-20948, Sensor_Motion:InvenSense_QFN-24_3x3mm_P0.4mm, symbol Sensor_Motion:ICM-20948
- C1: renamed from R3; symbol Device:R -> Device:C
- C2: value 0.1uF -> 10nF
- C7: renamed from C3; value 1uF -> 10uF
- J1: footprint Connector_JST:JST_XH_S2B-XH-A-1_1x02_P2.50mm_Horizontal -> Connector_JST:JST_PH_S2B-PH-K_1x02_P2.00mm_Horizontal
- J2: renamed from J6; footprint Connector_JST:JST_PH_S2B-PH-K_1x02_P2.00mm_Horizontal -> Connector_Molex:Molex_PicoBlade_53048-0210_1x02_P1.25mm_Horizontal
- J3: renamed from J10; footprint Connector_JST:JST_PH_S2B-PH-K_1x02_P2.00mm_Horizontal -> Connector_Molex:Molex_PicoBlade_53048-0210_1x02_P1.25mm_Horizontal
- J4: renamed from J7; footprint Connector_JST:JST_PH_S2B-PH-K_1x02_P2.00mm_Horizontal -> Connector_Molex:Molex_PicoBlade_53048-0210_1x02_P1.25mm_Horizontal
- J5: renamed from J11; footprint Connector_JST:JST_PH_S2B-PH-K_1x02_P2.00mm_Horizontal -> Connector_Molex:Molex_PicoBlade_53048-0210_1x02_P1.25mm_Horizontal
- J6: renamed from J4; footprint Connector_PinHeader_2.54mm:PinHeader_1x08_P2.54mm_Vertical_SMD_Pin1Right -> Connector_PinHeader_2.00mm:PinHeader_1x10_P2.00mm_Vertical_SMD_Pin1Right; symbol Connector_Generic:Conn_01x08 -> Connector_Generic:Conn_01x10
- J7: renamed from J5; footprint Connector_PinHeader_2.54mm:PinHeader_1x08_P2.54mm_Vertical_SMD_Pin1Right -> Connector_PinHeader_2.00mm:PinHeader_1x10_P2.00mm_Vertical_SMD_Pin1Right; symbol Connector_Generic:Conn_01x08 -> Connector_Generic:Conn_01x10
- U5: renamed from U4; value ME6211C33M5G-N -> ME6217C33M5G; symbol LDO:ME6211C33M5G-N -> LDO:ME6217C33M5G
- renumbered C13 to C10, C14 to C11, C15 to C12, C7 to C5, D8 to D7, D7 to D8, Q4 to Q3, Q3 to Q4, R5 to R10, R17 to R14, R18 to R15, R21 to R16, R19 to R17, R22 to R18, R24 to R19, R25 to R20, R26 to R21, R27 to R22, R28 to R23, R7 to R4, R8 to R5, R9 to R6, R10 to R7, R6 to R8, R4 to R9, U2 to U1, U1 to U2, U5 to U4
Connections:
- net PSRAM_CS is gone; now on net U1TXD: ESP1.29 (SD3)
- net +3V3: now also C2.2, C6.2, C9.2, C3.1, R3.2, U3.13 (VDD), U3.22 (~CS), U3.8 (VDDIO); no longer C2.1, C6.1, C9.1
- net EXT_IO1: now also J7.7 (Pin_7); no longer J7.8 (Pin_8)
- net GND: now also C2.1, C6.1, C9.1, J6.10 (Pin_10), J7.10 (Pin_10), C3.2, U3.11 (FSYNC), U3.18 (GND), U3.20 (GND), U3.9 (SDO/AD0); no longer C2.2, C6.2, C9.2, J6.4 (Pin_4), J7.5 (Pin_5)
- net I2C0_SCL: now also U3.23 (SCL/SCLK)
- net I2C0_SDA: now also U3.24 (SDA/SDI)
- net I2C1_SCL: now also J7.6 (Pin_6); no longer J7.7 (Pin_7)
- net I2C1_SDA: now also J7.5 (Pin_5); no longer J7.6 (Pin_6)
- net MPU_INT: now also R3.1, U3.12 (INT1)
- net VCC: now reaches U5.4 (VIN)
- net VCC: now also C7.1, D1.2 (A), D5.1 (K), Q1.2 (S), U5.1 (CE)
- net at C4.2: now also U3.10 (REGOUT)
- net U1RXD: now reaches ESP1.28 (SD2)
- net U1RXD: now also J6.4 (Pin_4)
- net AUX_SCL renamed U1TXD
- net AUX_SDA: no longer names the net of J6.6 (Pin_6)
- net BUZ_1: no longer names the net of J6.8 (Pin_8)
- net BUZ_2: no longer names the net of J6.7 (Pin_7)
- net SCLK: no longer names the net of ESP1.31 (CLK)
- net SIO0: no longer names the net of ESP1.33 (SD1)
- net SIO1: no longer names the net of ESP1.27 (IO17)
- net SIO2: no longer names the net of ESP1.32 (SD0)
- net SIO3: no longer names the net of ESP1.30 (CMD)
- net VDD_SIO: no longer names the net of ESP1.26 (VDD_SDIO_NC)
- removed net VSS: C7.1, D1.2 (A), D5.1 (K), Q1.2 (S), U5.1 (VIN), U5.3 (EN)
- no-connect marks 30 -> 27
Other:
- moved on the sheet: AE1, C10, C11, C12, C5, C6, C7, C8, C9, D5, D6, D7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

Commit message: .
Parts:
- J2, J3, J4, J5: footprint Connector_Molex:Molex_PicoBlade_53048-0210_1x02_P1.25mm_Horizontal -> Connector_Custom:MX1.25_2P
Changed lines of the file:
@@
 F 0 "J2" H 9400 1700 50  0000 L CNN
 F 1 "Conn_01x02" H 9300 1400 50  0000 L CNN
-F 2 "Connector_Molex:Molex_PicoBlade_53048-0210_1x02_P1.25mm_Horizontal" H 9450 1600 50  0001 C CNN
+F 2 "Connector_Custom:MX1.25_2P" H 9450 1600 50  0001 C CNN
 F 3 "~" H 9450 1600 50  0001 C CNN
 	1    9450 1600
@@
 F 0 "J3" H 9400 4100 50  0000 L CNN
 F 1 "Conn_01x02" H 9250 3800 50  0000 L CNN
-F 2 "Connector_Molex:Molex_PicoBlade_53048-0210_1x02_P1.25mm_Horizontal" H 9450 4000 50  0001 C CNN
+F 2 "Connector_Custom:MX1.25_2P" H 9450 4000 50  0001 C CNN
 F 3 "~" H 9450 4000 50  0001 C CNN
 	1    9450 4000
@@
 F 0 "J4" H 9400 6500 50  0000 L CNN
 F 1 "Conn_01x02" H 9300 6200 50  0000 L CNN
-F 2 "Connector_Molex:Molex_PicoBlade_53048-0210_1x02_P1.25mm_Horizontal" H 9450 6400 50  0001 C CNN
+F 2 "Connector_Custom:MX1.25_2P" H 9450 6400 50  0001 C CNN
 F 3 "~" H 9450 6400 50  0001 C CNN
 	1    9450 6400
@@
 F 0 "J5" H 9400 9050 50  0000 L CNN
 F 1 "Conn_01x02" H 9250 8750 50  0000 L CNN
-F 2 "Connector_Molex:Molex_PicoBlade_53048-0210_1x02_P1.25mm_Horizontal" H 9450 8950 50  0001 C CNN
+F 2 "Connector_Custom:MX1.25_2P" H 9450 8950 50  0001 C CNN
 F 3 "~" H 9450 8950 50  0001 C CNN
 	1    9450 8950

Commit message: .
Parts:
- U2: footprint Package_TO_SOT_SMD:SOT-363_SC-70-6 -> Package_TO_SOT_SMD:SOT-563
Changed lines of the file:
@@
 F 0 "U2" H 2450 3915 50  0000 C CNN
 F 1 "BC847BDW1T1G" H 2450 3824 50  0000 C CNN
-F 2 "Package_TO_SOT_SMD:SOT-363_SC-70-6" H 2450 3100 50  0001 C CNN
+F 2 "Package_TO_SOT_SMD:SOT-563" H 2450 3100 50  0001 C CNN
 F 3 "" H 2450 3500 50  0001 C CNN
 	1    2450 3500

Commit message: .
Parts:
- removed R3: 10K, Resistor_SMD:R_0402_1005Metric, symbol Device:R
- removed SW1: SW_MEC_5E, Button:SKSC_NO_HOLE, symbol Switch:SW_MEC_5E
- removed U3: ICM-20948, Sensor_Motion:InvenSense_QFN-24_3x3mm_P0.4mm, symbol Sensor_Motion:ICM-20948
- added J8, J9: Conn_01x08, Connector_Custom:1x10_P2.0, symbol Connector_Generic:Conn_01x10
- added R25: 10K, Resistor_SMD:R_0402_1005Metric, symbol Device:R
- added U3: MPU-9250, Sensor_Motion:InvenSense_QFN-24_3x3mm_P0.4mm, symbol Sensor_Motion:MPU-9250
- added U6: ESP-PSRAM32, Package_SO:SOIC-8_3.9x4.9mm_P1.27mm, symbol Memory_RAM:ESP-PSRAM32
- U2: footprint Package_TO_SOT_SMD:SOT-563 -> esp-drone:SOT-563
Connections:
- net MOT3 is gone; now on net MOT_3: Q4.1 (G), R17.1
- net MOT4 is gone; now on net MOT_4: Q5.1 (G), R18.1
- net +3V3: now also J7.1 (Pin_1), J8.1 (Pin_1), J9.1 (Pin_1), R25.1, U3.1 (RESV_VDDIO), U3.13 (VDD), U3.22 (~CS), U3.8 (VDDIO)
- net ADC_BAT: now also ESP1.5 (SENSOR_VP)
- net ESP_IO0: no longer C5.1
- net EXT_IO1: now also ESP1.28 (SD2), J6.6 (Pin_6), J8.6 (Pin_6); no longer J7.7 (Pin_7)
- net GND: now also C5.1, J8.10 (Pin_10), J9.10 (Pin_10), U3.11 (FSYNC), U3.18 (GND), U3.20 (RESV_GND), U3.9 (AD0/MISO), U6.4 (VSS); no longer C5.2
- net I2C0_SCL: now also ESP1.12 (IO32), U3.23 (SCL/SCLK); no longer J6.3 (Pin_3)
- net I2C0_SDA: now also ESP1.13 (IO33), U3.24 (SDA/MOSI); no longer J6.2 (Pin_2)
- net I2C1_SCL: now also ESP1.38 (IO19), J6.3 (Pin_3), J8.3 (Pin_3); no longer J7.6 (Pin_6)
- net I2C1_SDA: now also ESP1.39 (IO22), J6.2 (Pin_2), J8.2 (Pin_2); no longer J7.5 (Pin_5)
- net LED_BLE: now also ESP1.22 (IO2)
- net LED_GRN: now also ESP1.42 (IO21)
- net LED_RED: now also ESP1.8 (SENSOR_VN)
- net MOT_1: now also ESP1.36 (IO23)
- net MOT_2: now also ESP1.24 (IO4)
- net MPU_INT: now also ESP1.7 (SENSOR_CAPN), R25.2, U3.12 (INT)
- net SPI_CLK: now also ESP1.14 (IO25), J7.4 (Pin_4), J9.4 (Pin_4); no longer J7.3 (Pin_3)
- net SPI_CS0: now also ESP1.21 (IO15), J7.2 (Pin_2), J9.2 (Pin_2); no longer J7.1 (Pin_1)
- net SPI_MOSI: now also ESP1.20 (IO13), J7.3 (Pin_3), J9.3 (Pin_3); no longer J7.2 (Pin_2), J7.4 (Pin_4)
- net U1RXD: now also ESP1.34 (IO5), J6.5 (Pin_5), J8.5 (Pin_5); no longer ESP1.28 (SD2), J6.4 (Pin_4)
- net U1TXD: now also ESP1.35 (IO18), J6.4 (Pin_4), J8.4 (Pin_4); no longer ESP1.29 (SD3), J6.5 (Pin_5)
- net at U1.B5 (CC2): now also R11.1
- net at U1.B8 (SBU2): no longer R11.1
- net MOT_3: now reaches ESP1.15 (IO26)
- net U2RXD: now reaches ESP1.16 (IO27)
- net U2RXD: now also J7.8 (Pin_8), J9.8 (Pin_8)
- net U2TXD: now reaches ESP1.17 (IO14)
- net U2TXD: now also J7.9 (Pin_9), J9.9 (Pin_9)
- net SPI_MISO: now reaches ESP1.18 (IO12)
- net SPI_MISO: now also J7.5 (Pin_5), J9.5 (Pin_5)
- net EXT_IO2: now reaches ESP1.25 (IO16)
- net EXT_IO2: now also J6.7 (Pin_7), J8.7 (Pin_7)
- net VDD_SIO: now reaches ESP1.26 (VDD_SDIO_NC)
- net VDD_SIO: now also C5.2, U6.8 (VCC)
- net SIO1: now reaches ESP1.27 (IO17)
- net SIO1: now also U6.2 (SO/SIO)
- net SIO3: now reaches ESP1.30 (CMD)
- net SIO3: now also U6.7 (SIO3)
- net SCLK: now reaches ESP1.31 (CLK)
- net SCLK: now also U6.6 (SCLK)
- net SIO2: now reaches ESP1.32 (SD0)
- net SIO2: now also U6.3 (SIO2)
- net SIO0: now reaches ESP1.33 (SD1)
- net SIO0: now also U6.5 (SI/SIO)
- net MOT_4: now reaches ESP1.6 (SENSOR_CAPP)
- net at C4.2: now also U3.10 (REGOUT)
- net EXT_IO3: now reaches J6.8 (Pin_8)
- net EXT_IO3: now also J8.8 (Pin_8)
- net EXT_IO4: now reaches J6.9 (Pin_9)
- net EXT_IO4: now also J8.9 (Pin_9)
- new net EXT_IO5: J7.6 (Pin_6), J9.6 (Pin_6)
- new net EXT_IO6: J7.7 (Pin_7), J9.7 (Pin_7)
- new net PSRAM_CS: ESP1.29 (SD3), U6.1 (~CE)
- no-connect marks 27 -> 25
Other:
- moved on the sheet: C6, C7, C9, D5, Q1, R10, R11, R13, R9, U5
