File: esp-drone.kicad_pcb (KiCad board)
At the start: 2 copper layers, 58.3 x 58.3 mm, 3 parts, among them P1 CF_EXP_LEFT, P2 CF_EXP_RIGHT

Commit message: sch finish
Parts:
- removed EXP_ORIENTATION: VAL**, bitcraze:EXP_ORIENTATION
- removed P1: CF_EXP_LEFT, connectors:BF090-10-X-B2
- removed P2: CF_EXP_RIGHT, connectors:BF090-10-X-B2
Other:
- board size 58.3 x 58.3 mm -> 72.8 x 72.8 mm
- copper layers 2 -> 4
- net class Default: clearance 0.1524 -> 0.2; trace_width 0.2032 -> 0.25; via_dia 0.635 -> 0.8; via_drill 0.381 -> 0.4
- rule trace_clearance: 0.1524 -> 0.2
- rule trace_min: 0.1524 -> 0.2
- rule via_min_drill: 0.381 -> 0.3
- rule via_min_size: 0.635 -> 0.4

Commit message: .
Other:
- board size 72.8 x 72.8 mm -> 58.3 x 58.3 mm
Changed lines of the file:
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@@
   (general
     (thickness 1.6)
-    (drawings 32)
+    (drawings 54)
     (tracks 0)
     (zones 0)
@@
     (uvia_drill 0.1)
   )
-  (gr_arc (start 0 48.790367) (end 22.98097 25.809397) (angle -24.24756936) (layer Edge.Cuts) (width 0.2))
-  (gr_line (start -36.150834 33.322407) (end -25.809397 22.98097) (layer Edge.Cuts) (width 0.2))
-  (gr_line (start -33.322407 36.150834) (end -22.98097 25.809397) (layer Edge.Cuts) (width 0.2))
-  (gr_line (start 22.98097 25.809397) (end 33.322407 36.150834) (layer Edge.Cuts) (width 0.2))
-  (gr_line (start -33.322407 -36.150834) (end -22.98097 -25.809397) (layer Edge.Cuts) (width 0.2))
-  (gr_line (start 22.98097 -25.809397) (end 33.322407 -36.150834) (layer Edge.Cuts) (width 0.2))
-  (gr_line (start 25.809397 22.98097) (end 36.150834 33.322407) (layer Edge.Cuts) (width 0.2))
-  (gr_arc (start 0 48.790367) (end -11.515748 18.398962) (angle -24.24756936) (layer Edge.Cuts) (width 0.2))
-  (gr_line (start -36.150834 -33.322407) (end -25.809397 -22.98097) (layer Edge.Cuts) (width 0.2))
-  (gr_line (start 25.809397 -22.98097) (end 36.150834 -33.322407) (layer Edge.Cuts) (width 0.2))
-  (gr_arc (start 35.532115 33.941125) (end 36.150834 34.559843) (angle -90) (layer Edge.Cuts) (width 0.2))
-  (gr_arc (start -9.75 20.749999) (end -10.5 20.749999) (angle -90) (layer Edge.Cuts) (width 0.2))
-  (gr_arc (start -11.249999 19.100302) (end -10.499999 19.100302) (angle -110.7524306) (layer Edge.Cuts) (width 0.2))
-  (gr_arc (start -48.790367 0) (end -25.809397 22.98097) (angle -90) (layer Edge.Cuts) (width 0.2))
-  (gr_arc (start 35.532115 -33.941125) (end 36.150834 -33.322407) (angle -90) (layer Edge.Cuts) (width 0.2))
-  (gr_arc (start -35.532115 -33.941125) (end -36.150834 -34.559843) (angle -90) (layer Edge.Cuts) (width 0.2))
-  (gr_arc (start -33.941125 -35.532115) (end -33.322407 -36.150834) (angle -90) (layer Edge.Cuts) (width 0.2))
-  (gr_arc (start -35.532115 33.941125) (end -36.150834 33.322407) (angle -90) (layer Edge.Cuts) (width 0.2))
-  (gr_arc (start -33.941125 35.532115) (end -34.559843 36.150834) (angle -90) (layer Edge.Cuts) (width 0.2))
-  (gr_arc (start 9.75 20.75) (end 9.75 21.5) (angle -90) (layer Edge.Cuts) (width 0.2))
-  (gr_line (start 10.5 20.75) (end 10.5 19.100302) (layer Edge.Cuts) (width 0.2))
-  (gr_line (start 34.559843 -36.150834) (end 36.150834 -34.559843) (layer Edge.Cuts) (width 0.2))
-  (gr_line (start -10.5 20.749999) (end -10.5 19.100302) (layer Edge.Cuts) (width 0.2))
-  (gr_line (start -36.150834 -34.559843) (end -34.559843 -36.150834) (layer Edge.Cuts) (width 0.2))
-  (gr_line (start -9.75 21.499999) (end 9.75 21.5) (layer Edge.Cuts) (width 0.2))
-  (gr_line (start 36.150834 34.559843) (end 34.559843 36.150834) (layer Edge.Cuts) (width 0.2))
-  (gr_arc (start 0 -48.790367) (end -22.98097 -25.809397) (angle -90) (layer Edge.Cuts) (width 0.2))
-  (gr_arc (start 11.25 19.100302) (end 11.515748 18.398962) (angle -110.7524306) (layer Edge.Cuts) (width 0.2))
-  (gr_line (start -34.559843 36.150834) (end -36.150834 34.559843) (layer Edge.Cuts) (width 0.2))
-  (gr_arc (start 48.790367 0) (end 25.809397 -22.98097) (angle -90) (layer Edge.Cuts) (width 0.2))
-  (gr_arc (start 33.941125 35.532115) (end 33.322407 36.150834) (angle -90) (layer Edge.Cuts) (width 0.2))
-  (gr_arc (start 33.941125 -35.532115) (end 34.559843 -36.150834) (angle -90) (layer Edge.Cuts) (width 0.2))
+  (gr_arc (start 24.926386 -27.399594) (end 24.756735 -26.876413) (angle -125.9286164) (layer Edge.Cuts) (width 0.2))
+  (gr_arc (start 41.013498 0) (end 13.796612 3.935873) (angle -36.77324075) (layer Edge.Cuts) (width 0.2))
+  (gr_line (start -24.756735 26.876413) (end -19.444817 21.564832) (layer Edge.Cuts) (width 0.2))
+  (gr_arc (start 41.013498 0) (end 21.56868 -19.446055) (angle -36.77324075) (layer Edge.Cuts) (width 0.2))
+  (gr_arc (start -24.926386 27.399594) (end -24.756735 26.876413) (angle -125.9286164) (layer Edge.Cuts) (width 0.2))
+  (gr_line (start -28.992233 26.869135) (end -27.570831 25.447823) (layer Edge.Cuts) (width 0.2))
+  (gr_line (start -26.877988 24.755025) (end -21.56868 19.446055) (layer Edge.Cuts) (width 0.2))
+  (gr_line (start 25.449578 -27.569211) (end 26.87098 -28.990522) (layer Edge.Cuts) (width 0.2))
+  (gr_arc (start -41.013498 0) (end -21.56868 19.446055) (angle -22.3819565) (layer Edge.Cuts) (width 0.2))
+  (gr_line (start 19.444817 -21.564832) (end 24.756735 -26.876413) (layer Edge.Cuts) (width 0.2))
+  (gr_line (start -26.87098 28.990522) (end -25.449578 27.569211) (layer Edge.Cuts) (width 0.2))
+  (gr_line (start 15.513498 2.649999) (end 15.513498 -2.65) (layer Edge.Cuts) (width 0.2))
+  (gr_arc (start -16.021337 -7.168813) (end -16.517418 -8.584406) (angle -70.68749723) (layer Edge.Cuts) (width 0.2))
+  (gr_arc (start 14.913498 2.649999) (end 14.913498 3.249999) (angle -90) (layer Edge.Cuts) (width 0.2))
+  (gr_arc (start 0 -41.010888) (end -19.444817 -21.564832) (angle -89.99635326) (layer Edge.Cuts) (width 0.2))
+  (gr_arc (start -41.013498 0) (end -15.628883 -10.576923) (angle -22.38195842) (layer Edge.Cuts) (width 0.2))
+  (gr_line (start 19.444817 21.564832) (end 24.756735 26.876413) (layer Edge.Cuts) (width 0.2))
+  (gr_arc (start -27.40118 24.924642) (end -27.570831 25.447823) (angle -125.9286164) (layer Edge.Cuts) (width 0.2))
+  (gr_arc (start -17.013498 10) (end -15.628883 10.576923) (angle -93.30732713) (layer Edge.Cuts) (width 0.2))
+  (gr_line (start 21.56868 19.446055) (end 26.877988 24.755025) (layer Edge.Cuts) (width 0.2))
+  (gr_line (start 21.56868 -19.446055) (end 26.877988 -24.755025) (layer Edge.Cuts) (width 0.2))
+  (gr_line (start -28.992233 -26.869135) (end -27.570831 -25.447823) (layer Edge.Cuts) (width 0.2))
+  (gr_arc (start -17.013498 -10) (end -16.517418 -8.584406) (angle -93.30736218) (layer Edge.Cuts) (width 0.2))
+  (gr_line (start -17.521337 -7.168813) (end -17.521337 7.168814) (layer Edge.Cuts) (width 0.2))
+  (gr_line (start -24.756735 -26.876413) (end -19.444817 -21.564832) (layer Edge.Cuts) (width 0.2))
+  (gr_line (start 27.570831 -25.447823) (end 28.992233 -26.869135) (layer Edge.Cuts) (width 0.2))
+  (gr_line (start 14.913498 -3.25) (end 14.390435 -3.25) (layer Edge.Cuts) (width 0.2))
+  (gr_arc (start -16.021337 7.168813) (end -17.521337 7.168814) (angle -70.68751853) (layer Edge.Cuts) (width 0.2))
+  (gr_arc (start 27.40118 -24.924642) (end 27.570831 -25.447823) (angle -125.9286164) (layer Edge.Cuts) (width 0.2))
+  (gr_line (start 27.570831 25.447823) (end 28.992233 26.869135) (layer Edge.Cuts) (width 0.2))
+  (gr_arc (start 14.390435 -3.85) (end 13.796612 -3.935873) (angle -98.22858262) (layer Edge.Cuts) (width 0.2))
+  (gr_arc (start 14.913498 -2.65) (end 15.513498 -2.65) (angle -90) (layer Edge.Cuts) (width 0.2))
+  (gr_arc (start 14.390435 3.849999) (end 14.390435 3.249999) (angle -98.22858262) (layer Edge.Cuts) (width 0.2))
+  (gr_line (start -26.877988 -24.755025) (end -21.56868 -19.446055) (layer Edge.Cuts) (width 0.2))
+  (gr_arc (start -24.926386 -27.399594) (end -25.449578 -27.569211) (angle -125.9286164) (layer Edge.Cuts) (width 0.2))
+  (gr_line (start 25.449578 27.569211) (end 26.87098 28.990522) (layer Edge.Cuts) (width 0.2))
+  (gr_arc (start 27.40118 24.924642) (end 26.877988 24.755025) (angle -125.9286164) (layer Edge.Cuts) (width 0.2))
+  (gr_line (start 14.390435 3.249999) (end 14.913498 3.249999) (layer Edge.Cuts) (width 0.2))
+  (gr_line (start -26.87098 -28.990522) (end -25.449578 -27.569211) (layer Edge.Cuts) (width 0.2))
+  (gr_arc (start -27.40118 -24.924642) (end -26.877988 -24.755025) (angle -125.9286164) (layer Edge.Cuts) (width 0.2))
+  (gr_arc (start 24.926386 27.399594) (end 25.449578 27.569211) (angle -125.9286164) (layer Edge.Cuts) (width 0.2))
+  (gr_arc (start 0 41.010888) (end 19.444817 21.564832) (angle -89.99635326) (layer Edge.Cuts) (width 0.2))
+  (gr_arc (start -27.224522 -28.636958) (end -26.87098 -28.990522) (angle -90) (layer Edge.Cuts) (width 0.2))
+  (gr_arc (start -28.63869 -27.222699) (end -28.992255 -27.576241) (angle -90) (layer Edge.Cuts) (width 0.2))
+  (gr_arc (start 28.63869 -27.222699) (end 28.992233 -26.869135) (angle -90) (layer Edge.Cuts) (width 0.2))
+  (gr_arc (start 28.63869 27.222699) (end 28.992255 27.576241) (angle -90) (layer Edge.Cuts) (width 0.2))
+  (gr_line (start 28.992255 27.576241) (end 27.578087 28.9905) (layer Edge.Cuts) (width 0.2))
+  (gr_arc (start 27.224522 -28.636958) (end 27.578087 -28.9905) (angle -90) (layer Edge.Cuts) (width 0.2))
+  (gr_arc (start 27.224522 28.636958) (end 26.87098 28.990522) (angle -90) (layer Edge.Cuts) (width 0.2))
+  (gr_arc (start -27.224522 28.636958) (end -27.578087 28.9905) (angle -90) (layer Edge.Cuts) (width 0.2))
+  (gr_line (start 27.578087 -28.9905) (end 28.992255 -27.576241) (layer Edge.Cuts) (width 0.2))
+  (gr_arc (start -28.63869 27.222699) (end -28.992233 26.869135) (angle -90) (layer Edge.Cuts) (width 0.2))
+  (gr_line (start -27.578087 -28.9905) (end -28.992255 -27.576241) (layer Edge.Cuts) (width 0.2))
+  (gr_line (start -28.992255 27.576241) (end -27.578087 28.9905) (layer Edge.Cuts) (width 0.2))
 )

Commit message: .
Parts:
- added AE1: Antenna, Antenna:CA-C03, F.Cu at (15.0, 0.00)
- added C1: 10uF, Resistor_SMD:R_0402_1005Metric, F.Cu at (92.8, -2.30)
- added C10: 0.1uF, Capacitor_SMD:C_0402_1005Metric, F.Cu at (86.1, 13.2)
- added C11: 10uF, Capacitor_SMD:C_0402_1005Metric, F.Cu at (103.3, -3.54)
- added C12: 0.1uF, Capacitor_SMD:C_0402_1005Metric, F.Cu at (94.7, 6.71)
- added C2: 10nF, Capacitor_SMD:C_0402_1005Metric, F.Cu at (103.1, -1.21)
- added C3: 0.1uF, Capacitor_SMD:C_0402_1005Metric, F.Cu at (94.7, 4.74)
- added C4: 0.1uF, Capacitor_SMD:C_0402_1005Metric, F.Cu at (91.9, 8.69)
- added C5: 0.1uF, Capacitor_SMD:C_0402_1005Metric, F.Cu at (100.2, 0.78)
- added C6: 1uF, Capacitor_SMD:C_0402_1005Metric, F.Cu at (97.3, 2.77)
- added C7: 10uF, Capacitor_SMD:C_0402_1005Metric, F.Cu at (86.1, 15.2)
- added C8: 0.1uF, Capacitor_SMD:C_0402_1005Metric, F.Cu at (89.0, 11.3)
- added C9: 10uF, Capacitor_SMD:C_0402_1005Metric, F.Cu at (97.6, 4.74)
- added D1: LED-WHT, LED_SMD:LED_0402_1005Metric, F.Cu at (91.5, 0.74)
- added D2: LED-BLE, LED_SMD:LED_0402_1005Metric, F.Cu at (91.5, 2.73)
- added D3: LED-RED, LED_SMD:LED_0402_1005Metric, F.Cu at (97.5, -5.18)
- added D4: LED-GRN, LED_SMD:LED_0402_1005Metric, F.Cu at (97.5, -3.19)
- added D5: BAT60B, Diode_SMD:D_SOD-323, F.Cu at (69.9, 13.4)
- added D6: 1N4148WT, Diode_SMD:D_SOD-523, F.Cu at (11.8, 11.8)
- added D7: 1N4148WT, Diode_SMD:D_SOD-523, F.Cu at (-11.8, 11.8)
- added D8: 1N4148WT, Diode_SMD:D_SOD-523, F.Cu at (11.8, -11.8)
- added D9: 1N4148WT, Diode_SMD:D_SOD-523, F.Cu at (-11.8, -11.8)
- added ESP1: ESP32PICO_D4, SOC:ESP32_PICO_D4, F.Cu at (3.30, 3.94)
- added FB1: 330R at 100MHz, Resistor_SMD:R_0402_1005Metric, F.Cu at (103.0, -9.50)
- added J1: Conn_01x02, Connector_JST:JST_PH_S2B-PH-K_1x02_P2.00mm_Horizontal, F.Cu at (-13.0, 4.06)
- added J2: Conn_01x02, Connector_Custom:MX1.25_2P, B.Cu at (12.9, 12.9)
- added J3: Conn_01x02, Connector_Custom:MX1.25_2P, B.Cu at (-12.9, 12.9)
- added J4: Conn_01x02, Connector_Custom:MX1.25_2P, B.Cu at (12.9, -12.9)
- added J5: Conn_01x02, Connector_Custom:MX1.25_2P, B.Cu at (-12.9, -12.9)
- added J6: Conn_01x08, Connector_PinHeader_2.00mm:PinHeader_1x10_P2.00mm_Vertical_SMD_Pin1Right, F.Cu at (0.00, -11.0)
- added J7: Conn_01x08, Connector_PinHeader_2.00mm:PinHeader_1x10_P2.00mm_Vertical_SMD_Pin1Right, F.Cu at (0.00, 11.0)
- added Q1: AO3401A, Package_TO_SOT_SMD:SOT-23, F.Cu at (99.3, -8.45)
- added Q2: AO3400A, Package_TO_SOT_SMD:SOT-23, F.Cu at (14.7, 14.7)
- added Q3: AO3400A, Package_TO_SOT_SMD:SOT-23, F.Cu at (-14.7, 14.7)
- added Q4: AO3400A, Package_TO_SOT_SMD:SOT-23, F.Cu at (14.7, -14.7)
- added Q5: AO3400A, Package_TO_SOT_SMD:SOT-23, F.Cu at (-14.7, -14.7)
- added R1: 5.1K, Resistor_SMD:R_0402_1005Metric, F.Cu at (-9.21, -4.51)
- added R10: 82K, Resistor_SMD:R_0402_1005Metric, F.Cu at (105.9, -9.50)
- added R11: 5.1K, Resistor_SMD:R_0402_1005Metric, F.Cu at (-9.21, -5.52)
- added R12: 10K, Resistor_SMD:R_0402_1005Metric, F.Cu at (-9.21, -3.43)
- added R13: 82K, Resistor_SMD:R_0402_1005Metric, F.Cu at (86.0, 7.28)
- added R14: 200R, Resistor_SMD:R_0402_1005Metric, F.Cu at (89.0, 9.27)
- added R15: 10K, Resistor_SMD:R_0402_1005Metric, F.Cu at (16.5, 16.5)
- added R16: 10K, Resistor_SMD:R_0402_1005Metric, F.Cu at (-16.5, 16.5)
- added R17: 10K, Resistor_SMD:R_0402_1005Metric, F.Cu at (16.5, -16.5)
- added R18: 10K, Resistor_SMD:R_0402_1005Metric, F.Cu at (-16.5, -16.5)
- added R19: 10K, Resistor_SMD:R_0402_1005Metric, F.Cu at (100.3, -1.20)
- added R2: 10K, Resistor_SMD:R_0402_1005Metric, F.Cu at (83.2, 12.9)
- added R20: 10K, Resistor_SMD:R_0402_1005Metric, F.Cu at (105.9, -7.51)
- added R21: 10K, Resistor_SMD:R_0402_1005Metric, F.Cu at (86.1, 9.27)
- added R22: 10K, Resistor_SMD:R_0402_1005Metric, F.Cu at (100.4, -5.18)
- added R23: 10K, Resistor_SMD:R_0402_1005Metric, F.Cu at (88.9, 5.29)
- added R3: 10K, Resistor_SMD:R_0402_1005Metric, F.Cu at (94.4, -0.31)
- added R4: 10K, Resistor_SMD:R_0402_1005Metric, F.Cu at (94.4, 1.68)
- added R5: 2K, Resistor_SMD:R_0402_1005Metric, F.Cu at (86.0, 5.29)
- added R6: 3K, Resistor_SMD:R_0402_1005Metric, F.Cu at (100.4, -3.19)
- added R7: 10K, Resistor_SMD:R_0402_1005Metric, F.Cu at (97.3, -1.20)
- added R8: 10K, Resistor_SMD:R_0402_1005Metric, F.Cu at (91.8, 4.72)
- added R9: 82K, Resistor_SMD:R_0402_1005Metric, F.Cu at (88.9, 7.28)
- added SW1: SW_MEC_5E, Button:SKSC_NO_HOLE, F.Cu at (88.4, -2.91)
- added SW2: SW_MEC_5E, Button:SKSC_NO_HOLE, F.Cu at (100.1, -13.4)
- added U1: USB_C_16_PIN, Connector_USB:USB_C_Receptacle_HRO_TYPE-C-31-M-12, F.Cu at (-15.5, -3.56)
- added U2: BC847BDW1T1G, Package_TO_SOT_SMD:SOT-363_SC-70-6, F.Cu at (65.7, 13.9)
- added U3: ICM-20948, Sensor_Motion:InvenSense_QFN-24_3x3mm_P0.4mm, F.Cu at (2.79, -5.46)
- added U4: CP2102N-A01-GQFN28, Package_DFN_QFN:QFN-28-1EP_5x5mm_P0.5mm_EP3.35x3.35mm, F.Cu at (-6.99, 0.64)
- added U5: ME6217C33M5G, Package_TO_SOT_SMD:SOT-23-5, F.Cu at (-5.84, -5.21)
Routing:
- added copper zone on B.Cu, net (none)
- added copper zone on F.Cu, net GND
Other:
- outline, holes or cut-outs redrawn
- net class Default: clearance 0.2 -> 0.127; trace_width 0.25 -> 0.127; via_dia 0.8 -> 0.4; via_drill 0.4 -> 0.2
- rule trace_clearance: 0.2 -> 0.127
- rule trace_min: 0.2 -> 0.127
- rule via_min_drill: 0.3 -> 0.2

Commit message: .
Parts:
- U2: footprint Package_TO_SOT_SMD:SOT-363_SC-70-6 -> Package_TO_SOT_SMD:SOT-563
- moved U2 70.7 mm to (-4.51, 5.59), turned to 180 degrees
Changed lines of the file:
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@@
     (add_net VDD33_ESP)
+  )
+  (module Package_TO_SOT_SMD:SOT-563 (layer F.Cu)
+    (at -4.5085 5.588 180)
+    (descr SOT563)
+    (tags SOT-563)
+    (attr smd)
+    (fp_text reference U2 (at 0 -1.7) (layer F.SilkS)
+      (effects (font (size 1 1) (thickness 0.15)))
+    )
+    (fp_text value BC847BDW1T1G (at 0 1.75) (layer F.Fab)
+      (effects (font (size 1 1) (thickness 0.15)))
+    )
+    (fp_text user %R (at 0 0 90) (layer F.Fab)
+      (effects (font (size 0.4 0.4) (thickness 0.0625)))
+    )
+    (fp_line (start -0.65 -0.5) (end -0.3 -0.85) (layer F.Fab) (width 0.1))
+    (fp_line (start 0.65 0.9) (end -0.65 0.9) (layer F.SilkS) (width 0.12))
+    (fp_line (start -0.9 -0.9) (end 0.65 -0.9) (layer F.SilkS) (width 0.12))
+    (fp_line (start -0.65 -0.5) (end -0.65 0.85) (layer F.Fab) (width 0.1))
+    (fp_line (start -0.65 0.85) (end 0.65 0.85) (layer F.Fab) (width 0.1))
+    (fp_line (start 0.65 0.85) (end 0.65 -0.85) (layer F.Fab) (width 0.1))
+    (fp_line (start 0.65 -0.85) (end -0.3 -0.85) (layer F.Fab) (width 0.1))
+    (fp_line (start -1.35 -1.1) (end 1.35 -1.1) (layer F.CrtYd) (width 0.05))
+    (fp_line (start -1.35 -1.1) (end -1.35 1.1) (layer F.CrtYd) (width 0.05))
+    (fp_line (start 1.35 1.1) (end 1.35 -1.1) (layer F.CrtYd) (width 0.05))
+    (fp_line (start 1.35 1.1) (end -1.35 1.1) (layer F.CrtYd) (width 0.05))
+    (pad 5 smd rect (at 0.75 0 180) (size 0.7 0.4) (layers F.Cu F.Paste F.Mask)
+      (net 34 "Net-(R2-Pad1)"))
+    (pad 4 smd rect (at 0.75 0.5 180) (size 0.7 0.4) (layers F.Cu F.Paste F.Mask)
+      (net 37 CP_RTS))
+    (pad 2 smd rect (at -0.75 0 180) (size 0.7 0.4) (layers F.Cu F.Paste F.Mask)
+      (net 36 "Net-(R8-Pad2)"))
+    (pad 6 smd rect (at 0.75 -0.5 180) (size 0.7 0.4) (layers F.Cu F.Paste F.Mask)
+      (net 6 ESP_IO0))
+    (pad 3 smd rect (at -0.75 0.5 180) (size 0.7 0.4) (layers F.Cu F.Paste F.Mask)
+      (net 8 ESP_EN))
+    (pad 1 smd rect (at -0.75 -0.5 180) (size 0.7 0.4) (layers F.Cu F.Paste F.Mask)
+      (net 33 CP_DTR))
+    (model ${KISYS3DMOD}/Package_TO_SOT_SMD.3dshapes/SOT-563.wrl
+      (at (xyz 0 0 0))
+      (scale (xyz 1 1 1))
+      (rotate (xyz 0 0 0))
+    )
+  )
+  (module Antenna:CA-C03 (layer F.Cu)
+    (at 15.013498 0 90)
+    (fp_text reference AE1 (at 0 -3.048 90) (layer F.SilkS)
+      (effects (font (size 1 1) (thickness 0.15)))
+    )
+    (fp_text value Antenna (at 0 2.794 90) (layer F.Fab)
+      (effects (font (size 1 1) (thickness 0.15)))
+    )
+    (fp_line (start -6.65 -4.8) (end -6.65 4.8) (layer F.Fab) (width 0.12))
+    (fp_line (start 6.65 -4.8) (end 6.65 4.8) (layer F.Fab) (width 0.12))
+    (fp_line (start -6.65 4.8) (end 6.65 4.8) (layer F.Fab) (width 0.12))
+    (fp_line (start -6.65 -4.8) (end 6.65 -4.8) (layer F.Fab) (width 0.12))
+    (pad 1 smd roundrect (at -2.75 0 90) (size 0.8 1.8) (layers F.Cu F.Paste F.Mask) (roundrect_rratio 0.25)
+      (net 1 "Net-(AE1-Pad1)"))
+    (pad 2 smd roundrect (at 2.75 0 90) (size 0.8 1.8) (layers F.Cu F.Paste F.Mask) (roundrect_rratio 0.25))
+    (model ${KIPRJMOD}/CA-C03.step
+      (at (xyz 0 0 0))
+      (scale (xyz 1 1 1))
+      (rotate (xyz -90 0 0))
+    )
   )
   (module Connector_Custom:MX1.25_2P (layer B.Cu)
@@
     (pad 1 smd roundrect (at -1.5 -1) (size 0.55 0.2) (layers F.Cu F.Paste F.Mask) (roundrect_rratio 0.25))
     (model ${KISYS3DMOD}/Package_DFN_QFN.3dshapes/QFN-24_3x3mm_P0.4mm_EP1.7x1.54mm.wrl
-      (at (xyz 0 0 0))
-      (scale (xyz 1 1 1))
-      (rotate (xyz 0 0 0))
-    )
-  )
-  (module Package_TO_SOT_SMD:SOT-363_SC-70-6 (layer F.Cu)
-    (at 65.697 13.852)
-    (descr "SOT-363, SC-70-6")
-    (tags "SOT-363 SC-70-6")
-    (attr smd)
-    (fp_text reference U2 (at 0 -2) (layer F.SilkS)
-      (effects (font (size 1 1) (thickness 0.15)))
-    )
-    (fp_text value BC847BDW1T1G (at 0 2 180) (layer F.Fab)
-      (effects (font (size 1 1) (thickness 0.15)))
-    )
-    (fp_line (start 0.7 -1.16) (end -1.2 -1.16) (layer F.SilkS) (width 0.12))
-    (fp_line (start -0.7 1.16) (end 0.7 1.16) (layer F.SilkS) (width 0.12))
-    (fp_line (start 1.6 1.4) (end 1.6 -1.4) (layer F.CrtYd) (width 0.05))
-    (fp_line (start -1.6 -1.4) (end -1.6 1.4) (layer F.CrtYd) (width 0.05))
-    (fp_line (start -1.6 -1.4) (end 1.6 -1.4) (layer F.CrtYd) (width 0.05))
-    (fp_line (start 0.675 -1.1) (end -0.175 -1.1) (layer F.Fab) (width 0.1))
-    (fp_line (start -0.675 -0.6) (end -0.675 1.1) (layer F.Fab) (width 0.1))
-    (fp_line (start -1.6 1.4) (end 1.6 1.4) (layer F.CrtYd) (width 0.05))
-    (fp_line (start 0.675 -1.1) (end 0.675 1.1) (layer F.Fab) (width 0.1))
-    (fp_line (start 0.675 1.1) (end -0.675 1.1) (layer F.Fab) (width 0.1))
-    (fp_line (start -0.175 -1.1) (end -0.675 -0.6) (layer F.Fab) (width 0.1))
-    (fp_text user %R (at 0 0 90) (layer F.Fab)
-      (effects (font (size 0.5 0.5) (thickness 0.075)))
-    )
-    (pad 6 smd rect (at 0.95 -0.65) (size 0.65 0.4) (layers F.Cu F.Paste F.Mask)
-      (net 6 ESP_IO0))
-    (pad 4 smd rect (at 0.95 0.65) (size 0.65 0.4) (layers F.Cu F.Paste F.Mask)
-      (net 37 CP_RTS))
-    (pad 2 smd rect (at -0.95 0) (size 0.65 0.4) (layers F.Cu F.Paste F.Mask)
-      (net 36 "Net-(R8-Pad2)"))
-    (pad 5 smd rect (at 0.95 0) (size 0.65 0.4) (layers F.Cu F.Paste F.Mask)
-      (net 34 "Net-(R2-Pad1)"))
-    (pad 3 smd rect (at -0.95 0.65) (size 0.65 0.4) (layers F.Cu F.Paste F.Mask)
-      (net 8 ESP_EN))
-    (pad 1 smd rect (at -0.95 -0.65) (size 0.65 0.4) (layers F.Cu F.Paste F.Mask)
-      (net 33 CP_DTR))
-    (model ${KISYS3DMOD}/Package_TO_SOT_SMD.3dshapes/SOT-363_SC-70-6.wrl
       (at (xyz 0 0 0))
       (scale (xyz 1 1 1))
@@
     )
   )
-  (module Antenna:CA-C03 (layer F.Cu)
-    (at 15.013498 0 90)
-    (fp_text reference AE1 (at 0 -3.048 90) (layer F.SilkS)
-      (effects (font (size 1 1) (thickness 0.15)))
-    )
-    (fp_text value Antenna (at 0 2.794 90) (layer F.Fab)
-      (effects (font (size 1 1) (thickness 0.15)))
-    )
-    (fp_line (start -6.65 -4.8) (end -6.65 4.8) (layer F.Fab) (width 0.12))
-    (fp_line (start 6.65 -4.8) (end 6.65 4.8) (layer F.Fab) (width 0.12))
-    (fp_line (start -6.65 4.8) (end 6.65 4.8) (layer F.Fab) (width 0.12))
-    (fp_line (start -6.65 -4.8) (end 6.65 -4.8) (layer F.Fab) (width 0.12))
-    (pad 1 smd roundrect (at -2.75 0 90) (size 1.2 2) (layers F.Cu F.Paste F.Mask) (roundrect_rratio 0.25)
-      (net 1 "Net-(AE1-Pad1)"))
-    (pad 2 smd roundrect (at 2.75 0 90) (size 1.2 2) (layers F.Cu F.Paste F.Mask) (roundrect_rratio 0.25))
-    (model ${KIPRJMOD}/CA-C03.step
-      (at (xyz 0 0 0))
-      (scale (xyz 1 1 1))
-      (rotate (xyz -90 0 0))
-    )
-  )
