File: esp-drone.kicad_pcb (KiCad board)
At the start: 4 copper layers, 58.3 x 58.3 mm, 66 parts, among them J1 Conn_01x02, J2 Conn_01x02, J3 Conn_01x02, J4 Conn_01x02, J5 Conn_01x02, J6 Conn_01x08, J7 Conn_01x08, Q1 AO3401A, Q2 AO3400A, Q3 AO3400A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

Commit message: .
Parts:
- removed R3: 10K, Resistor_SMD:R_0402_1005Metric
- removed SW1: SW_MEC_5E, Button:SKSC_NO_HOLE
- added J8: Conn_01x08, Connector_Custom:1x10_P2.0, F.Cu at (0.00, 11.0)
- added J9: Conn_01x08, Connector_Custom:1x10_P2.0, F.Cu at (0.00, -11.0)
- added R25: 10K, Resistor_SMD:R_0402_1005Metric, F.Cu at (8.64, -7.37)
- added U6: ESP-PSRAM32, Package_SO:SOIC-8_3.9x4.9mm_P1.27mm, F.Cu at (-1.27, 5.33)
- U2: footprint Package_TO_SOT_SMD:SOT-563 -> esp-drone:SOT-563
- U3: value ICM-20948 -> MPU-9250
- moved R10 114.6 mm to (-7.49, 7.11), turned to 90 degrees
- moved R4 112.3 mm to (-16.5, -15.5), turned to 135 degrees
- moved Q1 109.1 mm to (-9.14, 3.81), turned to 180 degrees
- moved D1 108.4 mm to (-15.5, -16.5), turned to 315 degrees
- moved D2 107.9 mm to (-15.5, 16.5), turned to 45 degrees
- moved C5 106.5 mm to (-6.10, 7.11), turned to 270 degrees
- moved R19 105.7 mm to (-5.46, -0.64)
- moved C11 103.3 mm to (0.00, -2.03)
- moved C2 103.3 mm to (0.00, -7.11), turned to 180 degrees
- moved C1 103.2 mm to (-9.91, 7.11), turned to 270 degrees
- moved R5 103.0 mm to (-16.5, 15.5), turned to 225 degrees
- moved FB1 101.5 mm to (1.78, -2.29), turned to 90 degrees
- moved R8 101.2 mm to (-9.14, -2.03)
- moved C12 100.3 mm to (-5.46, 0.64), turned to 180 degrees
- moved R22 98.7 mm to (1.78, -4.57), turned to 90 degrees
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Connections:
- C5 pad 1: ESP_IO0 -> GND
- C5 pad 2: GND -> VDD_SIO
- D2 pad 2: (no net) -> LED_BLE
- D3 pad 2: (no net) -> LED_RED
- D4 pad 2: (no net) -> LED_GRN
- ESP1 pad 12: (no net) -> I2C0_SCL
- ESP1 pad 13: (no net) -> I2C0_SDA
- ESP1 pad 14: (no net) -> SPI_CLK
- ESP1 pad 15: (no net) -> MOT_3
- ESP1 pad 16: (no net) -> U2RXD
- ESP1 pad 17: (no net) -> U2TXD
- ESP1 pad 18: (no net) -> SPI_MISO
- ESP1 pad 20: (no net) -> SPI_MOSI
- ESP1 pad 21: (no net) -> SPI_CS0
- ESP1 pad 22: (no net) -> LED_BLE
- ESP1 pad 24: (no net) -> MOT_2
- ESP1 pad 25: (no net) -> EXT_IO2
- ESP1 pad 26: (no net) -> VDD_SIO
- ESP1 pad 27: (no net) -> SIO1
- ESP1 pad 28: U1RXD -> EXT_IO1
- ESP1 pad 29: U1TXD -> PSRAM_CS
- ESP1 pad 30: (no net) -> SIO3
- ESP1 pad 31: (no net) -> SCLK
- ESP1 pad 32: (no net) -> SIO2
- ESP1 pad 33: (no net) -> SIO0
- ESP1 pad 34: (no net) -> U1RXD
- ESP1 pad 35: (no net) -> U1TXD
- ESP1 pad 36: (no net) -> MOT_1
- ESP1 pad 38: (no net) -> I2C1_SCL
- ESP1 pad 39: (no net) -> I2C1_SDA
- ESP1 pad 42: (no net) -> LED_GRN
- ESP1 pad 5: (no net) -> ADC_BAT
- ESP1 pad 6: (no net) -> MOT_4
- ESP1 pad 7: (no net) -> MPU_INT
- ESP1 pad 8: (no net) -> LED_RED
- J6 pad 2: I2C0_SDA -> I2C1_SDA
- J6 pad 3: I2C0_SCL -> I2C1_SCL
- J6 pad 4: U1RXD -> U1TXD
- J6 pad 5: U1TXD -> U1RXD
- J6 pad 6: (no net) -> EXT_IO1
- J6 pad 7: (no net) -> EXT_IO2
- J6 pad 8: (no net) -> EXT_IO3
- J6 pad 9: (no net) -> EXT_IO4
- J7 pad 1: (no net) -> +3V3
- J7 pad 2: SPI_MOSI -> SPI_CS0
- J7 pad 3: (no net) -> SPI_MOSI
- J7 pad 4: SPI_MOSI -> SPI_CLK
- J7 pad 5: I2C1_SDA -> SPI_MISO
- J7 pad 6: I2C1_SCL -> EXT_IO5
- J7 pad 7: (no net) -> EXT_IO6
- J7 pad 8: (no net) -> U2RXD
- J7 pad 9: (no net) -> U2TXD
- Q4 pad 1: MOT3 -> MOT_3
- Q5 pad 1: MOT4 -> MOT_4
- R17 pad 1: MOT3 -> MOT_3
- R18 pad 1: MOT4 -> MOT_4
- U1 pad B5: (no net) -> Net-(R11-Pad1)
- U1 pad B8: Net-(R11-Pad1) -> (no net)
- U3 pad 1: (no net) -> +3V3
Routing:
- net +BATT: track 0.00 -> 99.1 mm
- net +3V3: track 0.00 -> 60.0 mm, vias 0 -> 4
- net VDD33_ESP: track 0.00 -> 44.3 mm, vias 0 -> 2
- net VCC: track 0.00 -> 35.8 mm, vias 0 -> 2
- net SPI_MOSI: track 0.00 -> 31.9 mm, vias 0 -> 1
- net ESP_EN: track 0.00 -> 30.4 mm, vias 0 -> 4
- net MOT_3: track 0.00 -> 28.5 mm, vias 0 -> 2
- net VBUS: track 0.00 -> 28.4 mm
- net LED_BLE: track 0.00 -> 25.7 mm, vias 0 -> 2
- net ADC_BAT: track 0.00 -> 24.1 mm, vias 0 -> 2
- net U2TXD: track 0.00 -> 21.9 mm, vias 0 -> 1
- net LED_RED: track 0.00 -> 21.8 mm, vias 0 -> 2
- net SPI_CS0: track 0.00 -> 21.1 mm, vias 0 -> 1
- net MOT_2: track 0.00 -> 20.3 mm, vias 0 -> 2
- net CP_RXD: track 0.00 -> 19.0 mm, vias 0 -> 2
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- added copper zone on B.Cu, net GND
- removed copper zone on B.Cu, net (none)
Other:
- outline, holes or cut-outs redrawn
- net class Default: trace_width 0.127 -> 0.1524
- rule trace_min: 0.127 -> 0.1524

Commit message: .
Parts:
- removed C5: 0.1uF, Capacitor_SMD:C_0402_1005Metric
- removed U6: ESP-PSRAM32, Package_SO:SOIC-8_3.9x4.9mm_P1.27mm
Connections:
- ESP1 pad 10: (no net) -> unconnected-(ESP1-Pad10)
- ESP1 pad 11: (no net) -> unconnected-(ESP1-Pad11)
- ESP1 pad 44: (no net) -> unconnected-(ESP1-Pad44)
- ESP1 pad 45: (no net) -> unconnected-(ESP1-Pad45)
- ESP1 pad 47: (no net) -> unconnected-(ESP1-Pad47)
- ESP1 pad 48: (no net) -> unconnected-(ESP1-Pad48)
- SW2 pad 2: (no net) -> unconnected-(SW2-Pad2)
- SW2 pad 3: (no net) -> unconnected-(SW2-Pad3)
- U1 pad A8: (no net) -> unconnected-(U1-PadA8)
- U1 pad B8: (no net) -> unconnected-(U1-PadB8)
- U3 pad 21: (no net) -> unconnected-(U3-Pad21)
- U3 pad 7: (no net) -> unconnected-(U3-Pad7)
- U4 pad 1: (no net) -> unconnected-(U4-Pad1)
- U4 pad 10: (no net) -> unconnected-(U4-Pad10)
- U4 pad 11: (no net) -> unconnected-(U4-Pad11)
- U4 pad 12: (no net) -> unconnected-(U4-Pad12)
- U4 pad 13: (no net) -> unconnected-(U4-Pad13)
- U4 pad 14: (no net) -> unconnected-(U4-Pad14)
- U4 pad 15: (no net) -> unconnected-(U4-Pad15)
- U4 pad 16: (no net) -> unconnected-(U4-Pad16)
- U4 pad 17: (no net) -> unconnected-(U4-Pad17)
- U4 pad 18: (no net) -> unconnected-(U4-Pad18)
- U4 pad 19: (no net) -> unconnected-(U4-Pad19)
- U4 pad 2: (no net) -> unconnected-(U4-Pad2)
- U4 pad 20: (no net) -> unconnected-(U4-Pad20)
- U4 pad 21: (no net) -> unconnected-(U4-Pad21)
- U4 pad 22: (no net) -> unconnected-(U4-Pad22)
- U4 pad 23: (no net) -> unconnected-(U4-Pad23)
- U4 pad 27: (no net) -> unconnected-(U4-Pad27)
- U4 pad 6: (no net) -> unconnected-(U4-Pad6)
- U5 pad 3: (no net) -> unconnected-(U5-Pad3)
Routing:
- net SIO2: track 17.5 -> 0.00 mm, vias 2 -> 0
- net SCLK: track 15.0 -> 0.00 mm, vias 2 -> 0
- net SIO0: track 14.6 -> 0.00 mm, vias 2 -> 0
- net SIO3: track 12.9 -> 0.00 mm, vias 2 -> 0
- net VDD_SIO: track 12.2 -> 0.00 mm
- net PSRAM_CS: track 8.92 -> 0.00 mm, vias 2 -> 0
- net SIO1: track 8.03 -> 0.00 mm, vias 2 -> 0
- net VBUS: track 28.4 -> 27.3 mm
- net +BATT: track 99.1 -> 98.1 mm
- net VDD33_ESP: track 44.3 -> 43.7 mm
Other:
- net class Default removed
